Commit message: update

File: urdf/turtlebot3_burger.gazebo.xacro (robot description, xacro)
@@ -50,8 +50,8 @@
       <commandTopic>cmd_vel</commandTopic>
       <odometryTopic>odom</odometryTopic>
-      <odometryFrame>$(arg frame_prefix)/odom</odometryFrame>
+      <odometryFrame>$(arg frame_prefix)odom</odometryFrame>
       <odometrySource>world</odometrySource>
       <publishOdomTF>true</publishOdomTF>
-      <robotBaseFrame>$(arg frame_prefix)/base_footprint</robotBaseFrame>
+      <robotBaseFrame>$(arg frame_prefix)base</robotBaseFrame>
       <publishWheelTF>false</publishWheelTF>
       <publishTf>true</publishTf>
@@ -72,5 +72,5 @@
       <alwaysOn>true</alwaysOn>
       <bodyName>imu_link</bodyName>
-      <frameName>$(arg frame_prefix)/imu_link</frameName>
+      <frameName>$(arg frame_prefix)imu_link</frameName>
       <topicName>imu</topicName>
       <serviceName>imu_service</serviceName>
@@ -126,5 +126,5 @@
       <plugin name="gazebo_ros_lds_lfcd_controller" filename="libgazebo_ros_laser.so">
         <topicName>scan</topicName>
-        <frameName>$(arg frame_prefix)/base_scan</frameName>
+        <frameName>$(arg frame_prefix)base_scan</frameName>
       </plugin>
     </sensor>

File: urdf/turtlebot3_burger.urdf.xacro (robot description, xacro)
@@ -5,9 +5,10 @@
   <xacro:arg name="use_laser_noise" default="true"/>
   <xacro:arg name="laser_range_max" default="3.5"/>
-  <xacro:include filename="$(find coverage_control)/urdf/common_properties.xacro"/>
-  <xacro:include filename="$(find coverage_control)/urdf/turtlebot3_burger.gazebo.xacro"/>
-  <link name="base_footprint"/>
+  <xacro:include filename="$(find tb3_coverage_control)/urdf/common_properties.xacro"/>
+  <xacro:include filename="$(find tb3_coverage_control)/urdf/turtlebot3_burger.gazebo.xacro"/>
+  <!--実機モードでmotive由来のframeとopencr由来のframe（base_footprint）の干渉を防ぐためframe名を変更する-->
+  <link name="base"/>
   <joint name="base_joint" type="fixed">
-    <parent link="base_footprint"/>
+    <parent link="base"/>
     <child link="base_link"/>
     <origin xyz="0.0 0.0 0.010" rpy="0 0 0"/>
